File: PCB/Mainboard/RC_Buggy.kicad_pcb (KiCad board)
At the start: 4 copper layers, 93.5 x 94.5 mm, 162 parts, among them J1 TYPE-C-31-M-12, J10 I2C, J11 Servo 0, J12 Servo 1, J13 PW_IO_bak, J14 PW_IO_bak, J15 Servo 4, J16 Servo 5, J17 Servo 2, J18 Servo 3, J19 Servo 6, J2 BME680, J20 Servo 7, J3 GPIO, J4 PW_5V, J5 PW_3V3, J6 Micro_SD_Card_Det_Hirose_DM3AT, J7 Stepper_1, J8 Stepper_2, J9 SPI, P1 TMC2209_Socket, P2 TMC2209_Socket, Q1 AON7262E, Q2 AON7262E, SW1 SW_Push, SW2 SW_Push, U1 ESP32-S3-WROOM-1, U10 TPS56637RPAR, U3 TPD4E05U06DQA, U4 TXS0108EPW, U5 PCA9685BS, U6 TPS62933, U7 TPS62933, U8 TPS56637RPAR, U9 TPS56637RPAR

Commit message: Added setup, read and get Command
Other:
- board text added: "Author: @THEFLOCKE"
Changed lines of the file:
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@@
 			(dashed_line_gap_ratio 3.000000)
 			(svgprecision 4)
-			(plotframeref no)
+			(plotframeref yes)
 			(mode 1)
 			(useauxorigin no)
@@
 			(pdf_back_fp_property_popups yes)
 			(pdf_metadata yes)
-			(pdf_single_document no)
+			(pdf_single_document yes)
 			(dxfpolygonmode yes)
 			(dxfimperialunits yes)
@@
 			(psnegative no)
 			(psa4output no)
-			(plot_black_and_white yes)
+			(plot_black_and_white no)
 			(sketchpadsonfab no)
 			(plotpadnumbers no)
@@
 			(crossoutdnponfab yes)
 			(subtractmaskfromsilk no)
-			(outputformat 1)
+			(outputformat 4)
 			(mirror no)
-			(drillshape 1)
+			(drillshape 0)
 			(scaleselection 1)
-			(outputdirectory "")
+			(outputdirectory "/Users/philipp/Downloads/KiCAD/")
 		)
 	)
@@
 		)
 	)
+	(gr_text "Author: @THEFLOCKE\n"
+		(at 250.3 196.35 0)
+		(layer "Cmts.User")
+		(effects
+			(font
+				(size 1.27 1.27)
+				(thickness 0.15875)
+			)
+		)
+	)
